File: untitled.kicad_sch (KiCad schematic)
At the start: 28 parts, among them J12 XT30UPB-M, J5 XT30UPB-M, SW6 SW_SPDT, U1 AMS1117-5.0, U2 AP62300TWU

Commit message: Updated
Parts:
- C15: value 10u -> 0.1u
- R12: value 10k -> 6.8k
- R3: value 1k -> 130
- R6: value 31.6k -> 33.2k
- R8: value 1k -> 10k
- R9: value 4.3k -> 51k
Changed lines of the file:
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@@
 			)
 		)
-		(property "Value" "10k"
+		(property "Value" "6.8k"
 			(at 52.07 100.3299 0)
 			(show_name no)
@@
 			)
 		)
-		(property "Value" "10u"
+		(property "Value" "0.1u"
 			(at 85.09 85.344 0)
 			(show_name no)
@@
 			)
 		)
-		(property "Value" "1k"
+		(property "Value" "130"
 			(at 158.75 43.18 90)
 			(show_name no)
@@
 			)
 		)
-		(property "Value" "31.6k"
+		(property "Value" "33.2k"
 			(at 96.52 88.8999 0)
 			(show_name no)
@@
 			)
 		)
-		(property "Value" "1k"
+		(property "Value" "10k"
 			(at 96.52 96.5199 0)
 			(show_name no)
@@
 			)
 		)
-		(property "Value" "4.3k"
+		(property "Value" "51k"
 			(at 52.07 92.7099 0)
 			(show_name no)
