File: untitledIC.kicad_sch (KiCad schematic)
At the start: 51 parts, among them J1 USB_C_Receptacle_USB2.0_14P, J10 Conn_01x20_MountingPin, J17 HC-05 Breakout Board, J2 Conn_01x04_Pin, J6 Conn_01x02_Pin, J8 Conn_01x02_Pin, SW10 SW_Push, SW11 SW_Push, SW12 SW_SPDT, SW5 Reset, SW7 Reset, SW9 SW_Push, U12 STM32F103C8Tx, U13 AMS1117-3.3, Y1 Crystal

Commit message: PCB
Parts:
- removed C22, C26: 100nF, Capacitor_SMD:C_0603_1608Metric_Pad1.08x0.95mm_HandSolder, symbol Device:C
- removed C24, C25: 10u, Capacitor_SMD:C_0603_1608Metric_Pad1.08x0.95mm_HandSolder, symbol Device:C
- removed C29: 100n, Capacitor_SMD:C_0603_1608Metric_Pad1.08x0.95mm_HandSolder, symbol Device:C_Small
- removed JP3: SolderJumper_2_Bridged, Jumper:SolderJumper-2_P1.3mm_Open_RoundedPad1.0x1.5mm, symbol Jumper:SolderJumper_2_Open
- removed R19: 100k, Resistor_SMD:R_0603_1608Metric_Pad0.98x0.95mm_HandSolder, symbol Device:R_US
- removed R21: 10k, Resistor_SMD:R_0603_1608Metric_Pad0.98x0.95mm_HandSolder, symbol Device:R_Small
- removed SW11: SW_Push, customs:Push button-fp, symbol Switch:SW_Push
- removed SW7: Reset, RESET:SW_TS09-63-25_CUD, symbol Switch:SW_Push
- removed U13: AMS1117-3.3, Package_TO_SOT_SMD:SOT-223-3_TabPin2, symbol Regulator_Linear:AMS1117-3.3
- added C40, C41: 0.01u, Capacitor_SMD:C_0603_1608Metric_Pad1.08x0.95mm_HandSolder, symbol Device:C_Small
- added J19: Conn_01x02_Socket, Connector_JST:JST_PH_B2B-PH-K_1x02_P2.00mm_Vertical, symbol Connector:Conn_01x02_Socket
- added SW1: SW_SPDT, Connector_PinHeader_2.00mm:PinHeader_1x03_P2.00mm_Vertical, symbol Switch:SW_SPDT
- D25, D26: footprint LED_THT:LED_D3.0mm -> LED_SMD:LED_0603_1608Metric_Pad1.05x0.95mm_HandSolder
- J1: footprint usb c vikram bhaiya:USB-C-16P -> CustomLibrary:USB-C-16P
- J2: footprint (none) -> Connector_PinHeader_2.00mm:PinHeader_1x04_P2.00mm_Vertical
- SW10, SW9: footprint customs:Push button-fp -> CustomLibrary:Push button-fp
- SW5: footprint RESET:SW_TS09-63-25_CUD -> CustomLibrary:Push button-fp
- TB2: footprint customs:TB6612 module -> CustomLibrary:TB6612 module
Connections:
- net AIN1_t is gone; now on net AIN1I: TB2.6 (AIN1)
- net AIN2_t is gone; now on net AIN2I: TB2.7 (AIN2)
- net BIN1_t is gone; now on net BIN1I: TB2.4 (BIN1)
- net BIN2_t is gone; now on net BIN2I: TB2.3 (BIN2)
- net MCU_RX is gone; now on net MCU_RXI: J17.4 (TXD)
- net MCU_TX is gone; now on net MCU_TXI: J17.5 (RXD)
- net Motor1+_t is gone; now on net Motor1+I: TB2.13 (M1Out+)
- net Motor1-_t is gone; now on net Motor1-I: TB2.12 (M1Out-)
- net Motor2+_t is gone; now on net Motor2+I: TB2.10 (M2Out+)
- net Motor2-_t is gone; now on net Motor2-I: TB2.11 (M2Out-)
- net PWMA_t is gone; now on net PWMAI: TB2.8 (PWMA)
- net PWMB_t is gone; now on net PWMBI: TB2.2 (PWMB)
- net GND: now also C40.2, C41.2, J19.1 (Pin_1), SW1.1 (A)
- net VDD: now also SW1.3 (C)
- net at R18.1: now also SW1.2 (B)
- net MCU_TXI: now reaches U12.21 (PB10)
- net MCU_RXI: now reaches U12.22 (PB11)
- net Button2I: now reaches U12.40 (PB4)
- net Button2I: now also SW10.2
- net ESC_PWMI: now reaches U12.41 (PB5)
- net ESC_PWMI: now also J19.2 (Pin_2)
- net AIN1 renamed AIN1I
- net AIN2 renamed AIN2I
- net BAT+ renamed BAT+I
- net BAT+_Driver renamed BAT+_DriverI
- net BAT+_DriverI: now also C40.1, C41.1
- net BAT_SNS renamed BAT_SNSI
- net BIN1 renamed BIN1I
- net BIN2 renamed BIN2I
- net BatteryLED renamed BatteryLEDI
- net Button1: no longer names the net of U12.20 (PB2)
- net Button1: no longer SW9.2
- net Button2 renamed Button1I
- net Button1I: now also SW9.2; no longer SW10.2
- net Button3: no longer names the net of U12.38 (PA15)
- net EN renamed ENI
- net Motor1+ renamed Motor1+I
- net Motor1- renamed Motor1-I
- net Motor2+ renamed Motor2+I
- net Motor2- renamed Motor2-I
- net PWMA renamed PWMAI
- net PWMB renamed PWMBI
- net SNSR1 renamed SNSR1I
- net SNSR2 renamed SNSR2I
- net SNSR3 renamed SNSR3I
- net SNSR4 renamed SNSR4I
- net SNSR5 renamed SNSR5I
- net SNSR6 renamed SNSR6I
- net SNSR7 renamed SNSR7I
- net SNSR8 renamed SNSR8I
- net SNSR9 renamed SNSR9I
- no-connect marks 14 -> 12
Other:
- note added: "ESC Signal"
- note added: "Motor Driver Decoupling"
- note removed: "USB STM 3.3"
- moved on the sheet: C10, C20, C21, C4, C5, C9, FB2

Commit message: Updated
Parts:
- R24: value 1k -> 130
Changed lines of the file:
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@@
 			)
 		)
-		(property "Value" "1k"
+		(property "Value" "130"
 			(at 252.73 146.05 90)
 			(show_name no)
