File: untitledPIC.kicad_sch (KiCad schematic)
At the start: 28 parts, among them J12 XT30UPB-M, J5 XT30UPB-M, SW6 SW_SPDT, U1 AMS1117-5.0, U2 AP62300TWU

Commit message: PCB
Parts:
- removed C11: 220u, Capacitor_THT:CP_Radial_D6.3mm_P2.50mm, symbol Device:C
- removed C12, C13, C14, C15, C7: 10u, Capacitor_SMD:C_0603_1608Metric_Pad1.08x0.95mm_HandSolder, symbol Device:C
- removed C16, C17: 22u, Capacitor_SMD:C_0603_1608Metric_Pad1.08x0.95mm_HandSolder, symbol Device:C
- removed C6: 0.1u, Capacitor_SMD:C_0603_1608Metric_Pad1.08x0.95mm_HandSolder, symbol Device:C
- removed D3: LED, LED_SMD:LED_0603_1608Metric_Pad1.05x0.95mm_HandSolder, symbol Device:LED
- removed D5: SS34, Diode_SMD:D_SMA_Handsoldering, symbol Diode:SS34
- removed F1: Polyfuse, Fuse:Fuse_0805_2012Metric_Pad1.15x1.40mm_HandSolder, symbol Device:Polyfuse
- removed F3: Fuse, Capacitor_SMD:C_1808_4520Metric, symbol Device:Fuse
- removed H1, H2, H3, H4: MountingHole, MountingHole:MountingHole_3mm, symbol Mechanical:MountingHole
- removed J12, J5: XT30UPB-M, Connector_AMASS:AMASS_XT30UPB-M_1x02_P5.0mm_Vertical, symbol customs:XT30UPB-M
- removed L1: 3.3u, Inductor_SMD:L_Sunlord_SWPA5040S, symbol Device:L
- removed R12: 10k, Resistor_SMD:R_0603_1608Metric_Pad0.98x0.95mm_HandSolder, symbol Device:R
- removed R3, R8: 1k, Resistor_SMD:R_0603_1608Metric_Pad0.98x0.95mm_HandSolder, symbol Device:R
- removed R6: 31.6k, Resistor_SMD:R_0603_1608Metric_Pad0.98x0.95mm_HandSolder, symbol Device:R
- removed R9: 4.3k, Resistor_SMD:R_0603_1608Metric_Pad0.98x0.95mm_HandSolder, symbol Device:R
- removed SW6: SW_SPDT, Button_Switch_THT:SW_Slide_SPDT_Angled_CK_OS102011MA1Q, symbol Switch:SW_SPDT
- removed U1: AMS1117-5.0, Package_TO_SOT_SMD:SOT-223-3_TabPin2, symbol Regulator_Linear:AMS1117-5.0
- removed U2: AP62300TWU, Package_TO_SOT_SMD:TSOT-23-6, symbol Regulator_Switching:AP62300TWU
- added C24, C25, C31, C32, C33, C35: 10u, Capacitor_SMD:C_0603_1608Metric_Pad1.08x0.95mm_HandSolder, symbol Device:C
- added C34: 220u, Capacitor_THT:CP_Radial_D6.3mm_P2.50mm, symbol Device:C
- added C36, C37: 22u, Capacitor_SMD:C_0603_1608Metric_Pad1.08x0.95mm_HandSolder, symbol Device:C
- added D27: SS34, Diode_SMD:D_SMA_Handsoldering, symbol Diode:SS34
- added D28: LED, LED_SMD:LED_0603_1608Metric_Pad1.05x0.95mm_HandSolder, symbol Device:LED
- added F4: Fuse, Capacitor_SMD:C_1808_4520Metric, symbol Device:Fuse
- added F5: Polyfuse, Fuse:Fuse_0805_2012Metric_Pad1.15x1.40mm_HandSolder, symbol Device:Polyfuse
- added H10, H11, H12, H9: MountingHole, MountingHole:MountingHole_3mm, symbol Mechanical:MountingHole
- added J13, J15: XT30UPB-M, Connector_AMASS:AMASS_XT30UPB-M_1x02_P5.0mm_Vertical, symbol customs:XT30UPB-M
- added JP3: SolderJumper_2_Bridged, Jumper:SolderJumper-2_P1.3mm_Open_RoundedPad1.0x1.5mm, symbol Jumper:SolderJumper_2_Open
- added L2: 3.3u, Inductor_SMD:L_Sunlord_SWPA5040S, symbol Device:L
- added R26: 4.3k, Resistor_SMD:R_0603_1608Metric_Pad0.98x0.95mm_HandSolder, symbol Device:R
- added R27: 10k, Resistor_SMD:R_0603_1608Metric_Pad0.98x0.95mm_HandSolder, symbol Device:R
- added R28: 31.6k, Resistor_SMD:R_0603_1608Metric_Pad0.98x0.95mm_HandSolder, symbol Device:R
- added R29, R30: 1k, Resistor_SMD:R_0603_1608Metric_Pad0.98x0.95mm_HandSolder, symbol Device:R
- added SW13: SW_SPDT, Button_Switch_THT:SW_Slide_SPDT_Angled_CK_OS102011MA1Q, symbol Switch:SW_SPDT
- added U13: AMS1117-3.3, Package_TO_SOT_SMD:SOT-223-3_TabPin2, symbol Regulator_Linear:AMS1117-3.3
- added U14: AMS1117-5.0, Package_TO_SOT_SMD:SOT-223-3_TabPin2, symbol Regulator_Linear:AMS1117-5.0
- added U15: AP62300TWU, Package_TO_SOT_SMD:TSOT-23-6, symbol Regulator_Switching:AP62300TWU
Connections:
- net +3.3V: now also C36.1, C37.1, JP3.2 (B), L2.2, R28.2, R30.1
- net +5V: now also C33.1, U14.2 (VO)
- net GND: now also C24.2, C25.2, C31.2, C32.1, C33.2, C34.2, C36.2, C37.2, D28.1 (K), J13.1 (N), J15.1 (N), R27.1, R29.1, U13.1 (GND), U14.1 (GND), U15.1 (GND)
- new net: R28.1, R29.2, U15.4 (FB)
- new net: C34.1, D27.1 (K), SW13.2 (B)
- new net: C35.1, L2.1, U15.2 (SW)
- new net: R26.1, R27.2, U15.5 (EN)
- new net: C35.2, U15.6 (BST)
- new net: D28.2 (A), R30.2
- new net: F4.2, J13.2 (P)
- new net BAT+I: C31.1, C32.2, R26.2, SW13.1 (A), U14.3 (VI), U15.3 (IN)
- new net ESC_POWI: D27.2 (A), F4.1, J15.2 (P)
- new net VBUS: C24.1, U13.3 (VI)
- new net VDD: C25.1, F5.1, JP3.1 (A), U13.2 (VO)
- new net VDD_STM: F5.2
Other:
- note added: "IC FUSE"
- note added: "USB STM 3.3"
- note removed: "DECOUPLING CAPACITORS"
- note removed: "Fuse"

Commit message: Updated
Parts:
- C35: value 10u -> 0.1u
- R26: value 4.3k -> 51k
- R27: value 10k -> 6.8k
- R28: value 31.6k -> 33.2k
- R29: value 1k -> 10k
- R30: value 1k -> 130
Changed lines of the file:
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@@
 			)
 		)
-		(property "Value" "31.6k"
+		(property "Value" "33.2k"
 			(at 99.06 87.6299 0)
 			(show_name no)
@@
 			)
 		)
-		(property "Value" "1k"
+		(property "Value" "10k"
 			(at 99.06 95.2499 0)
 			(show_name no)
@@
 			)
 		)
-		(property "Value" "1k"
+		(property "Value" "130"
 			(at 161.29 41.91 90)
 			(show_name no)
@@
 			)
 		)
-		(property "Value" "4.3k"
+		(property "Value" "51k"
 			(at 54.61 91.4399 0)
 			(show_name no)
@@
 			)
 		)
-		(property "Value" "10u"
+		(property "Value" "0.1u"
 			(at 87.63 84.074 0)
 			(show_name no)
@@
 			)
 		)
-		(property "Value" "10k"
+		(property "Value" "6.8k"
 			(at 54.61 99.0599 0)
 			(show_name no)
