File: LineFollowerGOAT.kicad_pcb (KiCad board)
At the start: 2 copper layers, 164.1 x 103.2 mm, 206 parts, among them J1 USB_C_Receptacle_USB2.0_14P, J10 Conn_01x20_MountingPin, J11 Conn_01x02_Pin, J12 XT30UPB-M, J13 XT30UPB-M, J15 XT30UPB-M, J16 HC-05 Breakout Board, J17 HC-05 Breakout Board, J18 Conn_01x02_Socket, J19 Conn_01x02_Socket, J2 Conn_01x04_Pin, J3 Conn_01x02_Pin, J4 Conn_01x02_Pin, J5 XT30UPB-M, J6 Conn_01x02_Pin, J7 Conn_01x20_MountingPin, J8 Conn_01x02_Pin, J9 Conn_01x20_MountingPin, SW1 SW_SPDT, SW10 SW_Push, SW12 SW_SPDT, SW13 SW_SPDT, SW2 SW_Push, SW3 SW_Push, SW5 Reset, SW6 SW_SPDT, SW8 SW_SPDT, SW9 SW_Push, U1 AMS1117-5.0, U10 TCRT5000L, U11 TCRT5000L, U12 STM32F103C8Tx, U13 AMS1117-3.3, U14 AMS1117-5.0, U15 AP62300TWU, U16 TCRT5000L, U17 TCRT5000L, U18 TCRT5000L, U2 AP62300TWU, U20 TCRT5000L, U21 TCRT5000L, U22 TCRT5000L, U23 74HC4067, U24 74HC4067, U27 TCRT5000L, U3 TCRT5000L, U4 TCRT5000L, U5 TCRT5000L, U6 TCRT5000L, U7 TCRT5000L, U8 TCRT5000L, U9 TCRT5000L, Y1 Crystal

Commit message: Edited silkscreen
Parts:
- added G***: LOGO, Robo Logo:robo_logo.pretty, B.Cu at (52.9, 112.1)
- moved R79 2.64 mm to (204.2, 114.6)
- moved R80 2.64 mm to (204.1, 123.8)
- moved R81 2.64 mm to (200.4, 122.9)
- moved U18 2.64 mm to (204.6, 119.2)
Routing:
- net GND: track 522.5 -> 529.4 mm
- net +3.3V: track 632.7 -> 635.1 mm
- net Q16: track 126.9 -> 129.2 mm
Other:
- board size 164.1 x 103.2 mm -> 164 x 103.2 mm
- board text added: "DESIGNED BY :"
- board text added: "L-V2.0"
- board text added: "RM 17 ELEC :) Nikunj | Jaishnu | | Tanya | Kapilmeet | Daivik |"
- board text added: "https://github.com/NikunSinghal"

Commit message: Fixed issues
Routing:
- net BAT+_DriverI: track 35.4 -> 33.7 mm
Changed lines of the file:
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@@
 			(outputformat 1)
 			(mirror no)
-			(drillshape 1)
+			(drillshape 0)
 			(scaleselection 1)
-			(outputdirectory "")
+			(outputdirectory "gerber/")
 		)
 	)
@@
 	)
 	(segment
-		(start 93.25 124.645)
-		(end 93.25 126.29)
-		(width 0.2)
-		(layer "F.Cu")
-		(net "VDD_STM")
-	)
-	(segment
 		(start 95.71991 127.99)
 		(end 95.9875 128.25759)
@@
 	)
 	(segment
+		(start 92.95 125.99)
+		(end 93.5375 126.5775)
+		(width 0.2)
+		(layer "F.Cu")
+		(net "VDD_STM")
+	)
+	(segment
 		(start 94.95 126.1025)
 		(end 96.45 126.1025)
@@
 	)
 	(segment
+		(start 93.27 124.575)
+		(end 92.95 124.895)
+		(width 0.2)
+		(layer "F.Cu")
+		(net "VDD_STM")
+	)
+	(segment
 		(start 95.9875 128.72241)
 		(end 95.16991 129.54)
@@
 	)
 	(segment
+		(start 92.95 124.895)
+		(end 92.95 125.99)
+		(width 0.2)
+		(layer "F.Cu")
+		(net "VDD_STM")
+	)
+	(segment
 		(start 95.16991 129.54)
 		(end 94.13009 129.54)
@@
 	)
 	(segment
-		(start 93.25 126.29)
-		(end 93.5375 126.5775)
-		(width 0.2)
-		(layer "F.Cu")
-		(net "VDD_STM")
-	)
-	(segment
 		(start 92.7 130.97009)
 		(end 92.7 132.465)
@@
 	(segment
 		(start 111.2 157.49)
-		(end 112.303 157.49)
+		(end 111.2 155.74)
 		(width 0.2)
 		(layer "F.Cu")
@@
 	)
 	(segment
-		(start 111.2 155.74)
-		(end 111.2 156.387)
+		(start 111.2 157.49)
+		(end 112.303 157.49)
 		(width 0.2)
 		(layer "F.Cu")
@@
 	)
 	(segment
-		(start 111.2 156.387)
+		(start 112.303 157.49)
 		(end 113.57 158.757)
 		(width 0.2)
@@
 	)
 	(segment
-		(start 112.303 157.49)
+		(start 113.57 158.18)
 		(end 113.57 158.757)
 		(width 0.2)
