File: LineFollowerGOAT.kicad_pcb (KiCad board)
At the start: 2 copper layers, 164 x 103.2 mm, 207 parts, among them J1 USB_C_Receptacle_USB2.0_14P, J10 Conn_01x20_MountingPin, J11 Conn_01x02_Pin, J12 XT30UPB-M, J13 XT30UPB-M, J15 XT30UPB-M, J16 HC-05 Breakout Board, J17 HC-05 Breakout Board, J18 Conn_01x02_Socket, J19 Conn_01x02_Socket, J2 Conn_01x04_Pin, J3 Conn_01x02_Pin, J4 Conn_01x02_Pin, J5 XT30UPB-M, J6 Conn_01x02_Pin, J7 Conn_01x20_MountingPin, J8 Conn_01x02_Pin, J9 Conn_01x20_MountingPin, SW1 SW_SPDT, SW10 SW_Push, SW12 SW_SPDT, SW13 SW_SPDT, SW2 SW_Push, SW3 SW_Push, SW5 Reset, SW6 SW_SPDT, SW8 SW_SPDT, SW9 SW_Push, U1 AMS1117-5.0, U10 TCRT5000L, U11 TCRT5000L, U12 STM32F103C8Tx, U13 AMS1117-3.3, U14 AMS1117-5.0, U15 AP62300TWU, U16 TCRT5000L, U17 TCRT5000L, U18 TCRT5000L, U2 AP62300TWU, U20 TCRT5000L, U21 TCRT5000L, U22 TCRT5000L, U23 74HC4067, U24 74HC4067, U27 TCRT5000L, U3 TCRT5000L, U4 TCRT5000L, U5 TCRT5000L, U6 TCRT5000L, U7 TCRT5000L, U8 TCRT5000L, U9 TCRT5000L, Y1 Crystal

Commit message: pad size
Routing:
- net +3.3V: track 635.1 -> 629.9 mm
- net VDD_STM: track 41.3 -> 42.9 mm
- net SNSR2I: track 10.7 -> 12.1 mm
- net SNSR1I: track 6.75 -> 7.96 mm
- net GND: track 527.2 -> 528.1 mm, vias 621 -> 620
- net Button2I: track 20.8 -> 21.6 mm
